File: Skanas_frekvences_noteiksana/Skanas_frekvences_noteiksana.kicad_pcb (KiCad board)
At the start: 2 copper layers, 109.4 x 36.4 mm, 30 parts, among them J1 USB_B_Mini, J2 AVR-ISP-6, SW1 SW_Push, U1 LM321, U2 ATmega328P-PU, U3 LCD-016N002L, Y1 Crystal

Commit message: Kursa_dabs
Parts:
- removed DS1: WC1602A, Connector_PinSocket_2.54mm:PinSocket_1x16_P2.54mm_Vertical
- removed REF**: Banana_Jack_1Pin, Connector:Banana_Jack_1Pin
- removed REF**: PinHeader_1x01_P2.54mm_Vertical, Connector_PinHeader_2.54mm:PinHeader_1x01_P2.54mm_Vertical
- removed REF**: Pin_D1.3mm_L11.0mm, Connector_Pin:Pin_D1.3mm_L11.0mm
- removed U3: LCD-016N002L, Display:WC1602A
- added ?: Pin_D1.0mm_L10.0mm, Connector_Pin:Pin_D1.0mm_L10.0mm, F.Cu at (215.7, 99.3)
- added ?: Pin_D1.0mm_L10.0mm, Connector_Pin:Pin_D1.0mm_L10.0mm, F.Cu at (215.7, 68.3)
- added ?: Pin_D1.0mm_L10.0mm, Connector_Pin:Pin_D1.0mm_L10.0mm, F.Cu at (140.7, 68.3)
- added ?: Pin_D1.0mm_L10.0mm, Connector_Pin:Pin_D1.0mm_L10.0mm, F.Cu at (140.7, 99.3)
- added C10: 100nF, Capacitor_THT:C_Disc_D3.8mm_W2.6mm_P2.50mm, F.Cu at (191.2, 86.3)
- added C9: 1nF, Capacitor_THT:C_Disc_D3.8mm_W2.6mm_P2.50mm, F.Cu at (188.7, 86.3)
- added J3: Connector for LCD, Connector_PinSocket_2.54mm:PinSocket_1x16_P2.54mm_Vertical, F.Cu at (146.2, 68.4)
- C1: value C -> 1uF
- C2, C3, C8: value C -> 100nF
- C4: value C -> 1nF
- C5, C7: value C -> 22pF
- C6: value C -> 0.01uF
- J2: footprint Connector_IDC:IDC-Header_2x03_P2.54mm_Vertical -> Connector_PinHeader_2.54mm:PinHeader_2x03_P2.54mm_Vertical
- L1: value INDUCTOR -> 10uH
- MK1: footprint Connector_PinSocket_2.54mm:PinSocket_1x02_P2.54mm_Vertical -> Skanas_frekvences_noteiksana:Microphone
- R1, R2: value R -> 1k
- R3, R4, R8: value R -> 10k
- R5: value R -> 220k
- R6: value R -> 1.5k
- R7: value R -> 220
- RV1: value R_POT -> 10k; footprint Potentiometer_THT:Potentiometer_Bourns_3266Y_Vertical -> Potentiometer_THT:Potentiometer_Runtron_RM-065_Vertical
- U1: value LM321 -> LM324N
- Y1: value Crystal -> 16MHz
- moved MK1 176.4 mm to (219.5, 77.7)
- moved R1 176.2 mm to (207.0, 82.6)
- moved R4 175.8 mm to (212.6, 82.6)
- moved J1 171.1 mm to (213.4, 91.0), turned to 90 degrees
- moved R3 164.9 mm to (201.6, 72.5), turned to 270 degrees
- moved R5 163.7 mm to (190.8, 82.8)
- moved R2 161.1 mm to (196.3, 72.6), turned to 270 degrees
- moved R6 153.2 mm to (185.3, 72.6), turned to 270 degrees
- moved U1 144.1 mm to (198.8, 89.3), turned to 270 degrees
- moved C1 141.6 mm to (200.5, 68.5)
- moved R7 138.2 mm to (171.6, 73.0), turned to 0 degrees
- moved L1 108.5 mm to (148.6, 76.6), turned to 0 degrees
- moved C6 102.8 mm to (181.4, 82.8), turned to 90 degrees
- moved C7 89.9 mm to (166.6, 90.8), turned to 180 degrees
- moved Y1 76.3 mm to (160.3, 96.6), turned to 0 degrees
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Connections:
- J1 pad 6: Net-(J1-Pad6) -> Earth
- U1 pad 1: Net-(R3-Pad2) -> Net-(R5-Pad2)
- U1 pad 11: (no net) -> Earth
- U1 pad 2: Earth -> Net-(R2-Pad2)
- U1 pad 3: Net-(R2-Pad2) -> Net-(R3-Pad2)
- U1 pad 4: Net-(R5-Pad2) -> VCC
- U1 pad 5: VCC -> (no net)
Routing:
- net Net-(J2-Pad4): track 0.00 -> 35.5 mm
- net Net-(J2-Pad1): track 0.00 -> 35.3 mm
- net Net-(C6-Pad1): track 0.00 -> 33.8 mm
- net Net-(J2-Pad3): track 0.00 -> 33.8 mm, vias 0 -> 1
- net Net-(J3-Pad11): track 0.00 -> 32.1 mm
- net Net-(R3-Pad2): track 0.00 -> 28.9 mm
- net RST: track 0.00 -> 26.0 mm
- net Earth: track 0.00 -> 25.7 mm, vias 0 -> 1
- net Net-(R5-Pad2): track 0.00 -> 25.5 mm
- net Net-(J3-Pad6): track 0.00 -> 22.2 mm
- net Net-(J3-Pad14): track 0.00 -> 22.2 mm
- net Net-(J3-Pad13): track 0.00 -> 22.2 mm
- net Net-(J3-Pad12): track 0.00 -> 22.2 mm
- net Net-(J3-Pad4): track 0.00 -> 21.2 mm
- net Net-(J3-Pad3): track 0.00 -> 19.3 mm
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- added copper zone on B.Cu, net Earth
- added copper zone on F.Cu, net VCC
Other:
- board size 109.4 x 36.4 mm -> 91 x 39.5 mm
- net class Power_Supply added: clearance 0.3, trace_width 0.3, via_dia 1, via_drill 0.6
