File: Skanas_frekvences_noteiksana/Skanas_frekvences_noteiksana.sch (KiCad schematic (older format))
At the start: 27 parts, among them J1 USB_B_Mini, J2 AVR-ISP-6, SW1 SW_Push, U1 LM321, U2 ATmega328P-PU, U3 LCD-016N002L, Y1 Crystal

Commit message: Kursa_dabs
Parts:
- removed DS1: WC1602A, Connector_PinSocket_2.54mm:PinSocket_1x16_P2.54mm_Vertical, symbol Display_Character:WC1602A
- removed U1: LM321, Package_DIP:DIP-14_W7.62mm, symbol Amplifier_Operational:LM321
- removed U3: LCD-016N002L, Display:WC1602A, symbol Display_Character:LCD-016N002L
- added C10: 100nF, Capacitor_THT:C_Disc_D3.8mm_W2.6mm_P2.50mm, symbol Device:C
- added C9: 1nF, Capacitor_THT:C_Disc_D3.8mm_W2.6mm_P2.50mm, symbol Device:C
- added J3: Connector for LCD, Connector_PinSocket_2.54mm:PinSocket_1x16_P2.54mm_Vertical, symbol Connector:Conn_01x16_Female
- added U1: LM324N, Package_DIP:DIP-14_W7.62mm, symbol Skanas_frekvences_noteiksana_amp:LM324N
- C1: value C -> 1uF
- C2, C3, C8: value C -> 100nF
- C4: value C -> 1nF
- C5, C7: value C -> 22pF
- C6: value C -> 0.01uF
- L1: value INDUCTOR -> 10uH
- MK1: footprint Connector_PinSocket_2.54mm:PinSocket_1x02_P2.54mm_Vertical -> Skanas_frekvences_noteiksana:Microphone
- R1, R2: value R -> 1k
- R3, R4, R8: value R -> 10k
- R5: value R -> 220k
- R6: value R -> 1.5k
- R7: value R -> 220
- RV1: value R_POT -> 10k; footprint Potentiometer_THT:Potentiometer_Bourns_3266Y_Vertical -> Potentiometer_THT:Potentiometer_Runtron_RM-065_Vertical
- Y1: value Crystal -> 16MHz
Connections:
- net Earth: now also J1.6 (Shield), C10.2, C9.2, J3.1 (Pin_1), J3.16 (Pin_16), J3.5 (Pin_5), U1.11 (V-)
- net VCC: now also C10.1, C9.1, J3.2 (Pin_2), U1.4 (V+)
- net at U2.6 (PD4): now also J3.11 (Pin_11)
- net at U2.11 (PD5): now also J3.12 (Pin_12)
- net at U2.12 (PD6): now also J3.13 (Pin_13)
- net at U2.13 (PD7): now also J3.14 (Pin_14)
- net at R7.2: now also J3.15 (Pin_15)
- net at RV1.2: now also J3.3 (Pin_3)
- net at R3.2, R4.1: now also U1.3 (+)
- net at R2.2, R5.1: now also U1.2 (-)
- net at R5.2, R6.1: now also U1.1
- net at U2.4 (PD2): now also J3.4 (Pin_4)
- net at U2.5 (PD3): now also J3.6 (Pin_6)
- no-connect marks 19 -> 18
Other:
- moved on the sheet: C1, C2, C3, C4, C6, C8, J1, J2, L1, MK1, R1, R2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

Commit message: Kursa_darbs
Parts:
- U1: symbol Skanas_frekvences_noteiksana_amp:LM324N -> Skanas_frekvences_noteiksana-rescue:LM324N-Skanas_frekvences_noteiksana_amp
Changed lines of the file:
@@
 	4210 3150 4640 3150
 $Comp
-L Skanas_frekvences_noteiksana_amp:LM324N U1
+L Skanas_frekvences_noteiksana-rescue:LM324N-Skanas_frekvences_noteiksana_amp U1
 U 1 1 5CF05886
 P 4890 3050
@@
 F 1 "LM324N" H 4920 2880 50  0000 L CNN
 F 2 "Package_DIP:DIP-14_W7.62mm" H 4740 3050 50  0001 C CNN
-F 3 "" H 4740 3050 50  0001 C CNN
+F 3 "http://www.farnell.com/datasheets/2281534.pdf" H 4740 3050 50  0001 C CNN
 	1    4890 3050
 	1    0    0    -1
